File: tenax.kicad_pcb (KiCad board)
At the start: 2 copper layers, 249 x 99.5 mm, 54 parts, among them J1 AudioJack4, J2 AudioJack4, SW1 SW_SPST, SW10 SW_SPST, SW11 SW_SPST, SW12 SW_SPST, SW13 SW_SPST, SW14 SW_SPST, SW15 SW_SPST, SW16 SW_SPST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

Commit message: teardrops
Routing:
- net TX_l: track 27.6 -> 26.8 mm
